Commit message: Fixed up TRINA to avoid excessive joint limits

File: data/robots/TRINA.urdf (robot description, URDF)
Before this commit: robot Cholera, 21 links, 20 joints
Joints:
- joint left_shoulder_upperarm: limit lower=-6.28 upper=6.28 effort=150 velocity=3.33 -> lower=-4.71 upper=1.57 effort=150 velocity=3.33
- joint left_upperarm_forearm: limit lower=-6.28 upper=6.28 effort=28 velocity=3.33 -> lower=-3.14 upper=3.14 effort=28 velocity=3.33
- joint right_shoulder_upperarm: limit lower=-6.28 upper=6.28 effort=150 velocity=3.33 -> lower=-1.57 upper=4.71 effort=150 velocity=3.33
- joint right_upperarm_forearm: limit lower=-6.28 upper=6.28 effort=28 velocity=3.33 -> lower=-3.14 upper=3.14 effort=28 velocity=3.33
